File: LSR_drone.kicad_sch (KiCad schematic)
At the start: 16 parts, among them CN2 XT30UPB-M, U10 L293D, U13 L293D, U14 DC Motor, U15 DC Motor, U16 DC Motor, U17 DC Motor, U18 ARDUINO_NANO, U5 LM7805-5V, U9 LM7805-5V

Commit message: stuff
Parts:
- renumbered A to A1
Changed lines of the file:
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@@
 		(on_board yes)
 		(dnp no)
-		(property "Reference" "#PWR?"
+		(property "Reference" "#PWR0112"
 			(at 66.04 82.55 0)
 			(effects
@@
 			(project ""
 				(path "/107e1f23-db6c-4b58-bf37-c9c4d63c378b"
-					(reference "#PWR?")
+					(reference "#PWR0112")
 					(unit 0)
 				)
@@
 		(on_board yes)
 		(dnp no)
-		(property "Reference" "#PWR?"
+		(property "Reference" "#PWR0101"
 			(at 64.77 142.24 0)
 			(effects
@@
 			(project ""
 				(path "/107e1f23-db6c-4b58-bf37-c9c4d63c378b"
-					(reference "#PWR?")
+					(reference "#PWR0101")
 					(unit 0)
 				)
@@
 		(on_board yes)
 		(dnp no)
-		(property "Reference" "#PWR?"
+		(property "Reference" "#PWR0108"
 			(at 212.09 128.27 0)
 			(effects
@@
 			(project ""
 				(path "/107e1f23-db6c-4b58-bf37-c9c4d63c378b"
-					(reference "#PWR?")
+					(reference "#PWR0108")
 					(unit 0)
 				)
@@
 		(on_board yes)
 		(dnp no)
-		(property "Reference" "#PWR?"
+		(property "Reference" "#PWR0113"
 			(at 54.61 60.96 0)
 			(effects
@@
 			(project ""
 				(path "/107e1f23-db6c-4b58-bf37-c9c4d63c378b"
-					(reference "#PWR?")
+					(reference "#PWR0113")
 					(unit 0)
 				)
@@
 		(on_board yes)
 		(dnp no)
-		(property "Reference" "#PWR?"
+		(property "Reference" "#PWR0104"
 			(at 53.34 116.84 0)
 			(effects
@@
 			(project ""
 				(path "/107e1f23-db6c-4b58-bf37-c9c4d63c378b"
-					(reference "#PWR?")
+					(reference "#PWR0104")
 					(unit 0)
 				)
@@
 		(on_board yes)
 		(dnp no)
-		(property "Reference" "#PWR?"
+		(property "Reference" "#PWR0103"
 			(at 62.23 127 0)
 			(effects
@@
 			(project ""
 				(path "/107e1f23-db6c-4b58-bf37-c9c4d63c378b"
-					(reference "#PWR?")
+					(reference "#PWR0103")
 					(unit 0)
 				)
@@
 		(on_board yes)
 		(dnp no)
-		(property "Reference" "#PWR?"
+		(property "Reference" "#PWR0110"
 			(at 161.29 29.21 0)
 			(effects
@@
 			(project ""
 				(path "/107e1f23-db6c-4b58-bf37-c9c4d63c378b"
-					(reference "#PWR?")
+					(reference "#PWR0110")
 					(unit 0)
 				)
@@
 		(on_board yes)
 		(dnp no)
-		(property "Reference" "#PWR?"
+		(property "Reference" "#PWR0105"
 			(at 85.09 93.98 0)
 			(effects
@@
 			(project ""
 				(path "/107e1f23-db6c-4b58-bf37-c9c4d63c378b"
-					(reference "#PWR?")
+					(reference "#PWR0105")
 					(unit 0)
 				)
@@
 		(on_board yes)
 		(dnp no)
-		(property "Reference" "#PWR?"
+		(property "Reference" "#PWR0107"
 			(at 177.8 53.34 0)
 			(effects
@@
 			(project ""
 				(path "/107e1f23-db6c-4b58-bf37-c9c4d63c378b"
-					(reference "#PWR?")
+					(reference "#PWR0107")
 					(unit 0)
 				)
@@
 		(on_board yes)
 		(dnp no)
-		(property "Reference" "#PWR?"
+		(property "Reference" "#PWR0102"
 			(at 82.55 154.94 0)
 			(effects
@@
 			(project ""
 				(path "/107e1f23-db6c-4b58-bf37-c9c4d63c378b"
-					(reference "#PWR?")
+					(reference "#PWR0102")
 					(unit 0)
 				)
@@
 		(on_board yes)
 		(dnp no)
-		(property "Reference" "#PWR?"
+		(property "Reference" "#PWR0111"
 			(at 63.5 71.12 0)
 			(effects
@@
 			(project ""
 				(path "/107e1f23-db6c-4b58-bf37-c9c4d63c378b"
-					(reference "#PWR?")
+					(reference "#PWR0111")
 					(unit 0)
 				)
@@
 		(on_board yes)
 		(dnp no)
-		(property "Reference" "#PWR?"
+		(property "Reference" "#PWR0106"
 			(at 193.04 50.8 0)
 			(effects
@@
 			(project ""
 				(path "/107e1f23-db6c-4b58-bf37-c9c4d63c378b"
-					(reference "#PWR?")
+					(reference "#PWR0106")
 					(unit 0)
 				)
@@
 		(on_board yes)
 		(dnp no)
-		(property "Reference" "A"
+		(property "Reference" "A1"
 			(at 145.161 -4.9911 0)
 			(effects
@@
 			(project ""
 				(path "/107e1f23-db6c-4b58-bf37-c9c4d63c378b"
-					(reference "A")
+					(reference "A1")
 					(unit 0)
 				)
@@
 		(on_board yes)
 		(dnp no)
-		(property "Reference" "#PWR?"
+		(property "Reference" "#PWR0109"
 			(at 212.09 114.3 0)
 			(effects
@@
 			(project ""
 				(path "/107e1f23-db6c-4b58-bf37-c9c4d63c378b"
-					(reference "#PWR?")
-					(unit 0)
-				)
+					(reference "#PWR0109")
+					(unit 0)
+				)
